File: test_boards/gallery/gallery.kicad_pcb (KiCad board)
At the start: 2 copper layers, 18 parts

Commit message: adding combo footprint for to-220, to-218, and to-247
Parts:
- removed the Val** at (22.9, 58.4)
- removed the Val** at (22.9, 66.0)
- added Val**: U***, TO-220_V_069B, F.Cu at (20.3, 58.4)
- added Val**: U***, TO-220_TO-218_TO-247_V_079B, F.Cu at (36.8, 58.4)

Commit message: tweaking pads
Parts:
- moved Q*** 32.1 mm to (22.9, 134.6)
- moved Val** 15.3 mm to (25.4, 68.6)
- moved Q*** 14.4 mm to (33.0, 134.6)
- moved U*** 7.62 mm to (91.4, 43.2)
- moved G5LA-1A 5.24 mm to (44.5, 101.6)
- moved G5LA-1 5.08 mm to (20.3, 101.6)
- moved U*** 5.08 mm to (66.0, 43.2)
- moved Q*** 2.54 mm to (33.0, 127.0)
- moved U*** 2.54 mm to (22.9, 127.0)
- moved U*** 2.54 mm to (48.3, 43.2)
- moved Val** 2.54 mm to (22.9, 58.4)

Commit message: layout tweaks for screenshots
Parts:
- moved U*** 5.08 mm to (43.2, 43.2)
- moved Q*** 2.54 mm to (33.0, 124.5)
- moved U*** 2.54 mm to (22.9, 124.5)
- moved U*** 2.54 mm to (30.5, 43.2)
- moved Q*** 2.54 mm to (22.9, 132.1)
- moved Q*** 2.54 mm to (33.0, 132.1)
- moved Val** 2.54 mm to (25.4, 66.0)
Changed lines of the file:
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@@
     (mod_text_size 1 1)
     (mod_text_width 0.15)
-    (pad_size 2.5 2.5)
-    (pad_drill 1.5)
+    (pad_size 2.0066 4.0132)
+    (pad_drill 1.4224)
     (pad_to_mask_clearance 0)
     (aux_axis_origin 0 0)
@@
     )
   )
-  (module pads (layer F.Cu)
-    (at 21.59 256.54)
-    (fp_text reference pads (at 2.54 -7.62) (layer F.SilkS) hide
-      (effects (font (size 1 1) (thickness 0.15)))
-    )
-    (fp_text value VAL** (at 10.16 -7.62) (layer F.SilkS) hide
-      (effects (font (size 1 1) (thickness 0.15)))
-    )
-    (fp_text user "(fits 0.01\" trace)" (at 6.35 6.35) (layer F.SilkS)
-      (effects (font (size 0.762 0.762) (thickness 0.1524)))
-    )
-    (fp_text user "(fits 0.02\" trace)" (at 6.35 -3.81) (layer F.SilkS)
-      (effects (font (size 0.762 0.762) (thickness 0.1524)))
-    )
-    (fp_text user "0.079\" pad, 0.050\" drill" (at 6.35 16.51) (layer F.SilkS)
-      (effects (font (size 0.762 0.762) (thickness 0.1524)))
-    )
-    (fp_text user "0.069\" pad, 0.040\" drill" (at 6.35 5.08) (layer F.SilkS)
-      (effects (font (size 0.762 0.762) (thickness 0.1524)))
-    )
-    (fp_text user "0.059\" pad, 0.032\" drill" (at 6.35 -5.08) (layer F.SilkS)
-      (effects (font (size 0.762 0.762) (thickness 0.1524)))
-    )
-    (pad 1 thru_hole oval (at 12.7 0) (size 1.4986 2.9464) (drill 0.8128)
-      (layers *.Cu *.Mask F.SilkS)
-    )
-    (pad 4 thru_hole rect (at 10.16 0) (size 1.4986 2.9464) (drill 0.8128)
-      (layers *.Cu *.Mask F.SilkS)
-    )
-    (pad 6 thru_hole oval (at 7.62 0) (size 1.4986 2.2098) (drill 0.8128 (offset 0 0.3683))
-      (layers *.Cu *.Mask F.SilkS)
-    )
-    (pad 7 thru_hole oval (at 2.54 0) (size 1.4986 1.4986) (drill 0.8128)
-      (layers *.Cu *.Mask F.SilkS)
-    )
-    (pad 8 thru_hole rect (at 5.08 0) (size 1.4986 2.2098) (drill 0.8128 (offset 0 0.3683))
-      (layers *.Cu *.Mask F.SilkS)
-    )
-    (pad 10 thru_hole rect (at 0 0) (size 1.4986 1.4986) (drill 0.8128)
-      (layers *.Cu *.Mask F.SilkS)
-    )
-    (pad 10 thru_hole oval (at 2.54 10.16) (size 1.7526 1.7526) (drill 1.016)
-      (layers *.Cu *.Mask F.SilkS)
-    )
-    (pad 11 thru_hole oval (at 7.62 10.16) (size 1.7526 2.6289) (drill 1.016 (offset 0 0.43815))
-      (layers *.Cu *.Mask F.SilkS)
-    )
-    (pad 12 thru_hole oval (at 12.7 10.16) (size 1.7526 3.5052) (drill 1.016)
-      (layers *.Cu *.Mask F.SilkS)
-    )
-    (pad 13 thru_hole rect (at 10.16 10.16) (size 1.7526 3.5052) (drill 1.016)
-      (layers *.Cu *.Mask F.SilkS)
-    )
-    (pad 14 thru_hole rect (at 5.08 10.16) (size 1.7526 2.6289) (drill 1.016 (offset 0 0.43815))
-      (layers *.Cu *.Mask F.SilkS)
-    )
-    (pad 15 thru_hole rect (at 0 10.16) (size 1.7526 1.7526) (drill 1.016)
-      (layers *.Cu *.Mask F.SilkS)
-    )
-    (pad 16 thru_hole rect (at 0 20.32) (size 2.0066 2.0066) (drill 1.27)
-      (layers *.Cu *.Mask F.SilkS)
-    )
-    (pad 17 thru_hole circle (at 2.54 20.32) (size 2.0066 2.0066) (drill 1.27)
-      (layers *.Cu *.Mask F.SilkS)
-    )
-    (pad 13 thru_hole rect (at 5.08 20.32) (size 2.0066 3.0099) (drill 1.27 (offset 0 0.50165))
-      (layers *.Cu *.Mask F.SilkS)
-    )
-    (pad 14 thru_hole oval (at 7.62 20.32) (size 2.0066 3.0099) (drill 1.27 (offset 0 0.50165))
-      (layers *.Cu *.Mask F.SilkS)
-    )
-    (pad 15 thru_hole rect (at 10.16 20.32) (size 2.0066 4.0132) (drill 1.27)
-      (layers *.Cu *.Mask F.SilkS)
-    )
-    (pad 16 thru_hole oval (at 12.7 20.32) (size 2.0066 4.0132) (drill 1.27)
-      (layers *.Cu *.Mask F.SilkS)
-    )
-  )
   (module R_AXIAL_0W25 (layer F.Cu)
     (at 20.32 22.86)
@@
   )
   (module DIP6 (layer F.Cu)
-    (at 33.02 43.18)
+    (at 30.48 43.18)
     (descr "6-lead DIP package")
     (tags DIP)
@@
   )
   (module DIP8 (layer F.Cu)
-    (at 48.26 43.18)
+    (at 43.18 43.18)
     (descr "8-lead DIP package")
     (tags DIP)
@@
   )
   (module TO-220_TO-218_TO-247_V_079B (layer F.Cu)
-    (at 25.4 68.58)
+    (at 25.4 66.04)
     (descr "TO-220, TO-218, and TO-247 vertical, 079B pads")
     (tags "TR TO220")
@@
   )
   (module TO-92_Q (layer F.Cu)
-    (at 33.02 127)
+    (at 33.02 124.46)
     (descr "TO-92 Transistor")
     (tags DEV)
@@
   )
   (module TO-92_U (layer F.Cu)
-    (at 22.86 127)
+    (at 22.86 124.46)
     (descr "TO-92 Integrated Circuit")
     (tags DEV)
@@
   )
   (module TO-92_Q_CBE (layer F.Cu)
-    (at 22.86 134.62)
+    (at 22.86 132.08)
     (descr "TO-92 Transistor, CBE pinout")
     (tags DEV)
@@
   )
   (module TO-92_Q_EBC (layer F.Cu)
-    (at 33.02 134.62)
+    (at 33.02 132.08)
     (descr "TO-92 Transistor, EBC pinout")
     (tags DEV)
@@
       (layers *.Cu *.Mask F.SilkS)
     )
+  )
+  (module pads (layer F.Cu)
+    (at 21.59 256.54)
+    (fp_text reference pads (at 2.54 -7.62) (layer F.SilkS) hide
+      (effects (font (size 1 1) (thickness 0.15)))
+    )
+    (fp_text value VAL** (at 10.16 -7.62) (layer F.SilkS) hide
+      (effects (font (size 1 1) (thickness 0.15)))
+    )
+    (fp_text user "(fits 0.01\" trace)" (at 6.35 6.35) (layer F.SilkS)
+      (effects (font (size 0.762 0.762) (thickness 0.1524)))
+    )
+    (fp_text user "(fits 0.02\" trace)" (at 6.35 -3.81) (layer F.SilkS)
+      (effects (font (size 0.762 0.762) (thickness 0.1524)))
+    )
+    (fp_text user "0.079\" pad, 0.056\" drill" (at 6.35 16.51) (layer F.SilkS)
+      (effects (font (size 0.762 0.762) (thickness 0.1524)))
+    )
+    (fp_text user "0.069\" pad, 0.040\" drill" (at 6.35 5.08) (layer F.SilkS)
+      (effects (font (size 0.762 0.762) (thickness 0.1524)))
+    )
+    (fp_text user "0.059\" pad, 0.032\" drill" (at 6.35 -5.08) (layer F.SilkS)
+      (effects (font (size 0.762 0.762) (thickness 0.1524)))
+    )
+    (pad 1 thru_hole oval (at 12.7 0) (size 1.4986 2.9464) (drill 0.8128)
+      (layers *.Cu *.Mask F.SilkS)
+    )
+    (pad 4 thru_hole rect (at 10.16 0) (size 1.4986 2.9464) (drill 0.8128)
+      (layers *.Cu *.Mask F.SilkS)
+    )
+    (pad 6 thru_hole oval (at 7.62 0) (size 1.4986 2.2098) (drill 0.8128 (offset 0 0.3683))
+      (layers *.Cu *.Mask F.SilkS)
+    )
+    (pad 7 thru_hole oval (at 2.54 0) (size 1.4986 1.4986) (drill 0.8128)
+      (layers *.Cu *.Mask F.SilkS)
+    )
+    (pad 8 thru_hole rect (at 5.08 0) (size 1.4986 2.2098) (drill 0.8128 (offset 0 0.3683))
+      (layers *.Cu *.Mask F.SilkS)
+    )
+    (pad 10 thru_hole rect (at 0 0) (size 1.4986 1.4986) (drill 0.8128)
+      (layers *.Cu *.Mask F.SilkS)
+    )
+    (pad 10 thru_hole oval (at 2.54 10.16) (size 1.7526 1.7526) (drill 1.016)
+      (layers *.Cu *.Mask F.SilkS)
+    )
+    (pad 11 thru_hole oval (at 7.62 10.16) (size 1.7526 2.6289) (drill 1.016 (offset 0 0.43815))
+      (layers *.Cu *.Mask F.SilkS)
+    )
+    (pad 12 thru_hole oval (at 12.7 10.16) (size 1.7526 3.5052) (drill 1.016)
+      (layers *.Cu *.Mask F.SilkS)
+    )
+    (pad 13 thru_hole rect (at 10.16 10.16) (size 1.7526 3.5052) (drill 1.016)
+      (layers *.Cu *.Mask F.SilkS)
+    )
+    (pad 14 thru_hole rect (at 5.08 10.16) (size 1.7526 2.6289) (drill 1.016 (offset 0 0.43815))
+      (layers *.Cu *.Mask F.SilkS)
+    )
+    (pad 15 thru_hole rect (at 0 10.16) (size 1.7526 1.7526) (drill 1.016)
+      (layers *.Cu *.Mask F.SilkS)
+    )
+    (pad 16 thru_hole rect (at 0 20.32) (size 2.0066 2.0066) (drill 1.4224)
+      (layers *.Cu *.Mask F.SilkS)
+    )
+    (pad 17 thru_hole circle (at 2.54 20.32) (size 2.0066 2.0066) (drill 1.4224)
+      (layers *.Cu *.Mask F.SilkS)
+    )
+    (pad 13 thru_hole rect (at 5.08 20.32) (size 2.0066 3.0099) (drill 1.4224 (offset 0 0.50165))
+      (layers *.Cu *.Mask F.SilkS)
+    )
+    (pad 14 thru_hole oval (at 7.62 20.32) (size 2.0066 3.0099) (drill 1.4224 (offset 0 0.50165))
+      (layers *.Cu *.Mask F.SilkS)
+    )
+    (pad 15 thru_hole rect (at 10.16 20.32) (size 2.0066 4.0132) (drill 1.4224)
+      (layers *.Cu *.Mask F.SilkS)
+    )
+    (pad 16 thru_hole oval (at 12.7 20.32) (size 2.0066 4.0132) (drill 1.4224)
+      (layers *.Cu *.Mask F.SilkS)
+    )

Commit message: tweaking relays, adding dc barrel jacks
Parts:
- added CON***: BARREL_JACK, BARREL_JACK_21x55, F.Cu at (34.3, 149.9)
Other:
- board text added: "connectors_PL"
Changed lines of the file:
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@@
     (area 17.142178 16.28 401.217201 279.357448)
     (thickness 1.6)
-    (drawings 7)
+    (drawings 8)
     (tracks 22)
     (zones 0)
-    (modules 18)
+    (modules 19)
     (nets 1)
   )
@@
     (mod_text_size 1 1)
     (mod_text_width 0.15)
-    (pad_size 2.0066 4.0132)
-    (pad_drill 1.4224)
+    (pad_size 4.064 4.064)
+    (pad_drill 3.048)
     (pad_to_mask_clearance 0)
     (aux_axis_origin 0 0)
@@
     )
   )
+  (module BARREL_JACK_21x55 (layer F.Cu)
+    (at 34.29 149.86)
+    (descr "DC Barrel Jack, 2.1x5.5mm")
+    (tags "Power Jack")
+    (path PWR-Jack)
+    (fp_text reference CON*** (at -7.62 5.461) (layer F.SilkS)
+      (effects (font (size 0.762 0.762) (thickness 0.1524)))
+    )
+    (fp_text value BARREL_JACK (at -4.445 -5.334) (layer F.SilkS) hide
+      (effects (font (size 1.016 1.016) (thickness 0.2032)))
+    )
+    (fp_text user 2.1x5.5mm (at -2.667 -3.556) (layer F.SilkS)
+      (effects (font (size 0.762 0.762) (thickness 0.1524)))
+    )
+    (fp_line (start -10.1981 -4.50088) (end -10.1981 4.50088) (layer F.SilkS) (width 0.381))
+    (fp_line (start -13.69822 -4.50088) (end -13.69822 4.50088) (layer F.SilkS) (width 0.381))
+    (fp_line (start -13.69822 4.50088) (end 0.80264 4.50088) (layer F.SilkS) (width 0.381))
+    (fp_line (start 0.80264 4.50088) (end 0.80264 -4.50088) (layer F.SilkS) (width 0.381))
+    (fp_line (start 0.80264 -4.50088) (end -13.69822 -4.50088) (layer F.SilkS) (width 0.381))
+    (pad 1 thru_hole rect (at 0 0) (size 4.064 4.064) (drill 3.048)
+      (layers *.Cu *.Mask F.SilkS)
+    )
+    (pad 2 thru_hole circle (at -5.969 0) (size 4.064 4.064) (drill 3.048)
+      (layers *.Cu *.Mask F.SilkS)
+    )
+    (pad 3 thru_hole circle (at -3.048 4.699) (size 4.064 4.064) (drill 3.048)
+      (layers *.Cu *.Mask F.SilkS)
+    )
+  )
+  (gr_text connectors_PL (at 17.78 140.97) (layer F.SilkS)
+    (effects (font (size 1.5 1.5) (thickness 0.3)) (justify left))
+  )
   (gr_text transistors_PL (at 17.78 119.38) (layer F.SilkS)

Commit message: updating M3 mounting hole
Parts:
- moved H*** 1.27 mm to (326.4, 30.5)
Changed lines of the file:
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@@
     (add_net "")
-  )
-  (module hole_M3 (layer F.Cu)
-    (at 325.12 30.48)
-    (descr "M3 mounting hole")
-    (path 1pin)
-    (fp_text reference H*** (at 0 -3.048) (layer F.SilkS) hide
-      (effects (font (size 1.016 1.016) (thickness 0.254)))
-    )
-    (fp_text value Val** (at 0 2.794) (layer F.SilkS) hide
-      (effects (font (size 1.016 1.016) (thickness 0.254)))
-    )
-    (fp_circle (center 0 0) (end 0 3.2) (layer F.SilkS) (width 0.15))
-    (pad 1 thru_hole circle (at 0 0) (size 6 6) (drill 3.2)
-      (layers *.Cu *.Mask F.SilkS)
-    )
   )
   (module 530002B02500G (layer F.Cu)
@@
       (layers *.Cu *.Mask F.SilkS)
     )
+  )
+  (module hole_M3 (layer F.Cu)
+    (at 326.39 30.48)
+    (descr "M3 mounting hole")
+    (path 1pin)
+    (fp_text reference H*** (at 0 -3.048) (layer F.SilkS) hide
+      (effects (font (size 1.016 1.016) (thickness 0.254)))
+    )
+    (fp_text value Val** (at 0 2.794) (layer F.SilkS) hide
+      (effects (font (size 1.016 1.016) (thickness 0.254)))
+    )
+    (fp_circle (center 0 0) (end 4.5 0) (layer F.SilkS) (width 0.15))
+    (pad 1 thru_hole circle (at 0 0) (size 6 6) (drill 3.2)
+      (layers *.Cu *.Mask F.SilkS)
+    )

Commit message: adding vertical resistor.  adding 2.5x5.5mm barrel jack.
Parts:
- added CON***: BARREL_JACK, BARREL_JACK_25x55, F.Cu at (54.6, 149.9)
- added R***: VAL*, R_AXIAL_0W25_V, F.Cu at (35.6, 22.9)
Changed lines of the file:
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@@
     (tracks 22)
     (zones 0)
-    (modules 19)
+    (modules 21)
     (nets 1)
   )
@@
     (mod_text_size 1 1)
     (mod_text_width 0.15)
-    (pad_size 4.064 4.064)
-    (pad_drill 3.048)
+    (pad_size 2.2479 1.4986)
+    (pad_drill 0.8128)
     (pad_to_mask_clearance 0)
     (aux_axis_origin 0 0)
@@
     )
   )
+  (module BARREL_JACK_25x55 (layer F.Cu)
+    (at 54.61 149.86)
+    (descr "DC Barrel Jack, 2.5x5.5mm")
+    (tags "Power Jack")
+    (path PWR-Jack)
+    (fp_text reference CON*** (at -7.62 5.461) (layer F.SilkS)
+      (effects (font (size 0.762 0.762) (thickness 0.1524)))
+    )
+    (fp_text value BARREL_JACK (at -4.445 -5.334) (layer F.SilkS) hide
+      (effects (font (size 1.016 1.016) (thickness 0.2032)))
+    )
+    (fp_text user 2.5x5.5mm (at -2.667 -3.556) (layer F.SilkS)
+      (effects (font (size 0.762 0.762) (thickness 0.1524)))
+    )
+    (fp_line (start -10.1981 -4.50088) (end -10.1981 4.50088) (layer F.SilkS) (width 0.381))
+    (fp_line (start -13.69822 -4.50088) (end -13.69822 4.50088) (layer F.SilkS) (width 0.381))
+    (fp_line (start -13.69822 4.50088) (end 0.80264 4.50088) (layer F.SilkS) (width 0.381))
+    (fp_line (start 0.80264 4.50088) (end 0.80264 -4.50088) (layer F.SilkS) (width 0.381))
+    (fp_line (start 0.80264 -4.50088) (end -13.69822 -4.50088) (layer F.SilkS) (width 0.381))
+    (pad 1 thru_hole rect (at 0 0) (size 4.064 4.064) (drill 3.048)
+      (layers *.Cu *.Mask F.SilkS)
+    )
+    (pad 2 thru_hole circle (at -5.969 0) (size 4.064 4.064) (drill 3.048)
+      (layers *.Cu *.Mask F.SilkS)
+    )
+    (pad 3 thru_hole circle (at -3.048 4.699) (size 4.064 4.064) (drill 3.048)
+      (layers *.Cu *.Mask F.SilkS)
+    )
+  )
+  (module R_AXIAL_0W25_V (layer F.Cu)
+    (at 35.56 22.86)
+    (descr "1/4W resistor, vertical")
+    (tags R)
+    (autoplace_cost90 10)
+    (autoplace_cost180 10)
+    (fp_text reference R*** (at 1.27 -2.159) (layer F.SilkS)
+      (effects (font (size 0.762 0.762) (thickness 0.1524)))
+    )
+    (fp_text value VAL* (at 1.27 2.286) (layer F.SilkS) hide
+      (effects (font (size 0.762 0.762) (thickness 0.1524)))
+    )
+    (fp_circle (center 0 0) (end 1.27 0) (layer F.SilkS) (width 0.3048))
+    (fp_line (start 0 0) (end 2.54 0) (layer F.SilkS) (width 0.3048))
+    (pad 1 thru_hole oval (at 0 0) (size 2.2479 1.4986) (drill 0.8128 (offset -0.37465 0))
+      (layers *.Cu *.Mask F.SilkS)
+    )
+    (pad 2 thru_hole oval (at 2.54 0) (size 2.2479 1.4986) (drill 0.8128 (offset 0.37465 0))
+      (layers *.Cu *.Mask F.SilkS)
+    )
+    (model discret/verti_resistor.wrl
+      (at (xyz 0 0 0))
+      (scale (xyz 1 1 1))
+      (rotate (xyz 0 0 0))
+    )
+  )

Commit message: adding banana jack
Parts:
- added Banana_A: VAL**, Banana_A, F.Cu at (68.6, 149.9)
Changed lines of the file:
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@@
     (tracks 22)
     (zones 0)
-    (modules 21)
+    (modules 22)
     (nets 1)
   )
@@
     (mod_text_size 1 1)
     (mod_text_width 0.15)
-    (pad_size 2.2479 1.4986)
-    (pad_drill 0.8128)
+    (pad_size 9.144 9.144)
+    (pad_drill 6.096)
     (pad_to_mask_clearance 0)
     (aux_axis_origin 0 0)
@@
     )
   )
+  (module Banana_A (layer F.Cu)
+    (at 68.58 149.86)
+    (fp_text reference Banana_A (at 0 6.096) (layer F.SilkS) hide
+      (effects (font (size 0.762 0.762) (thickness 0.1524)))
+    )
+    (fp_text value VAL** (at 0 -6.096) (layer F.SilkS)
+      (effects (font (size 0.762 0.762) (thickness 0.1524)))
+    )
+    (fp_circle (center 0 0) (end 5.334 0) (layer F.SilkS) (width 0.3048))
+    (pad 1 thru_hole circle (at 0 0) (size 9.144 9.144) (drill 6.096)
+      (layers *.Cu *.Mask F.SilkS)
+    )
+  )
