File: test_boards/gallery/gallery.sch (KiCad schematic (older format))
At the start: 37 parts, among them CON101 BARREL_JACK, K101 RELAY_1_FORM_A, K102 RELAY_1_FORM_C, Q101 NPN_EBC, Q102 PNP_EBC, Q103 NPN_CBE, Q104 PNP_CBE, Q105 2N3904, Q106 2N3906, Q107 BC550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

Commit message: adding 7812 regulator.  updating line thickness of to-220 footprints.
Parts:
- added U?: 7812, ~, symbol 7812
Other:
- moved on the sheet: U105, U106
Changed lines of the file:
@@
 Sheet 1 1
 Title ""
-Date "23 mar 2014"
+Date "20 apr 2014"
 Rev ""
 Comp ""
@@
 L LM317 U105
 U 1 1 532A69C4
-P 2550 6500
-F 0 "U105" H 2350 6660 40  0000 L BNN
-F 1 "LM317" H 2750 6330 40  0000 R TNN
-F 2 "~" H 2550 6500 60  0000 C CNN
-F 3 "~" H 2550 6500 60  0000 C CNN
-	1    2550 6500
-	1    0    0    -1
-$EndComp
-$Comp
-L LM337 U106
-U 1 1 532A69D3
 P 3300 6500
-F 0 "U106" H 3100 6660 40  0000 L BNN
-F 1 "LM337" H 3500 6330 40  0000 R TNN
+F 0 "U105" H 3100 6660 40  0000 L BNN
+F 1 "LM317" H 3500 6330 40  0000 R TNN
 F 2 "~" H 3300 6500 60  0000 C CNN
 F 3 "~" H 3300 6500 60  0000 C CNN
 	1    3300 6500
+	1    0    0    -1
+$EndComp
+$Comp
+L LM337 U106
+U 1 1 532A69D3
+P 4050 6500
+F 0 "U106" H 3850 6660 40  0000 L BNN
+F 1 "LM337" H 4250 6330 40  0000 R TNN
+F 2 "~" H 4050 6500 60  0000 C CNN
+F 3 "~" H 4050 6500 60  0000 C CNN
+	1    4050 6500
 	1    0    0    -1
 $EndComp
@@
 	1    0    0    -1
 $EndComp
+$Comp
+L 7812 U?
+U 1 1 535372C9
+P 2550 6500
+F 0 "U?" H 2350 6660 40  0000 L BNN
+F 1 "7812" H 2750 6330 40  0000 R TNN
+F 2 "~" H 2550 6500 60  0000 C CNN
+F 3 "~" H 2550 6500 60  0000 C CNN
+	1    2550 6500
+	1    0    0    -1
+$EndComp

Commit message: saving project
Parts:
- added U?: XR-2206, ~, symbol XR-2206
Other:
- note added: "analog_ICs_PL"
Changed lines of the file:
@@
 EESchema Schematic File Version 2
+LIBS:analog_ICs_PL
 LIBS:diodes_PL
 LIBS:switches_PL
@@
 Sheet 1 1
 Title ""
-Date "20 apr 2014"
+Date "4 may 2014"
 Rev ""
 Comp ""
@@
 	1    0    0    -1
 $EndComp
+Text Notes 3500 1650 0    60   ~ 0
+analog_ICs_PL
+$Comp
+L XR-2206 U?
+U 1 1 5366539C
+P 3950 2450
+F 0 "U?" H 3675 3100 60  0000 C CNN
+F 1 "XR-2206" H 4225 1775 60  0000 C CNN
+F 2 "~" H 3950 2450 60  0000 C CNN
+F 3 "~" H 3950 2450 60  0000 C CNN
+	1    3950 2450
+	1    0    0    -1
+$EndComp

Commit message: updating gallery
Parts:
- added C?: C_FILM, ~, symbol C_FILM
Changed lines of the file:
@@
+	1    0    0    -1
+$EndComp
+$Comp
+L C_FILM C?
+U 1 1 5366B32A
+P 4600 1000
+F 0 "C?" H 4620 1060 30  0000 L BNN
+F 1 "C_FILM" H 4620 940 30  0000 L TNN
+F 2 "~" H 4638 850 30  0000 C CNN
+F 3 "~" H 4600 1000 60  0000 C CNN
+	1    4600 1000
 	1    0    0    -1
 $EndComp

Commit message: pulling in 4P4C connector and symbol.
Parts:
- added J?: 4P4C, ~, symbol 4P4C
Changed lines of the file:
@@
 Sheet 1 1
 Title ""
-Date "4 may 2014"
+Date "4 jun 2014"
 Rev ""
 Comp ""
@@
 L AMMETER_H DS101
 U 1 1 532A694E
-P 1700 5500
-F 0 "DS101" H 1750 5650 40  0000 L CNN
-F 1 "AMMETER_H" H 2550 5100 40  0000 R CNN
-F 2 "~" H 2530 5900 60  0000 C CNN
-F 3 "~" H 2530 5900 60  0000 C CNN
-	1    1700 5500
+P 2900 5500
+F 0 "DS101" H 2950 5650 40  0000 L CNN
+F 1 "AMMETER_H" H 3750 5100 40  0000 R CNN
+F 2 "~" H 3730 5900 60  0000 C CNN
+F 3 "~" H 3730 5900 60  0000 C CNN
+	1    2900 5500
 	1    0    0    -1
 $EndComp
@@
 L AMMETER_V DS102
 U 1 1 532A695D
-P 2850 5500
-F 0 "DS102" H 2900 5650 40  0000 L CNN
-F 1 "AMMETER_V" H 3700 5100 40  0000 R CNN
-F 2 "~" H 3680 5900 60  0000 C CNN
-F 3 "~" H 3680 5900 60  0000 C CNN
-	1    2850 5500
+P 4050 5500
+F 0 "DS102" H 4100 5650 40  0000 L CNN
+F 1 "AMMETER_V" H 4900 5100 40  0000 R CNN
+F 2 "~" H 4880 5900 60  0000 C CNN
+F 3 "~" H 4880 5900 60  0000 C CNN
+	1    4050 5500
 	1    0    0    -1
 $EndComp
@@
 L VOLTMETER DS103
 U 1 1 532A696C
-P 4000 5500
-F 0 "DS103" H 4050 5650 40  0000 L CNN
-F 1 "VOLTMETER" H 4850 5100 40  0000 R CNN
-F 2 "~" H 4830 5900 60  0000 C CNN
-F 3 "~" H 4830 5900 60  0000 C CNN
-	1    4000 5500
-	1    0    0    -1
-$EndComp
-Text Notes 1650 5250 0    60   ~ 0
+P 5200 5500
+F 0 "DS103" H 5250 5650 40  0000 L CNN
+F 1 "VOLTMETER" H 6050 5100 40  0000 R CNN
+F 2 "~" H 6030 5900 60  0000 C CNN
+F 3 "~" H 6030 5900 60  0000 C CNN
+	1    5200 5500
+	1    0    0    -1
+$EndComp
+Text Notes 2850 5250 0    60   ~ 0
 displays_PL
 $Comp
@@
 	1    0    0    -1
 $EndComp
+$Comp
+L 4P4C J?
+U 1 1 538E6894
+P 2000 5650
+F 0 "J?" H 2200 6150 60  0000 C CNN
+F 1 "4P4C" H 1850 6150 60  0000 C CNN
+F 2 "~" H 2000 5650 60  0000 C CNN
+F 3 "~" H 2000 5650 60  0000 C CNN
+	1    2000 5650
+	1    0    0    -1
+$EndComp
